File: pcb/belt.kicad_sch (KiCad schematic)
At the start: 4 parts

Commit message: mostly finished schematic
Other:
- note added: "TODO: - Add test points - De-page schematic"
- note removed: "TODO: - Add decoupling caps - Add indicator LEDs"
- moved on the sheet: H1, H2, H3, H4
Changed lines of the file:
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@@
   (title_block
     (title "Basic Electronics Learning Toolkit")
-    (date "2023-12-31")
+    (date "2024-01-02")
     (rev "0.2")
     (company "Rice Eclipse")
@@
     (stroke (width 0) (type default))
   )
-  (text "TODO: \n- Add decoupling caps\n- Add indicator LEDs" (at 100.33 124.46 0)
+  (text_box "Mounting"
+    (at 190.5 63.5 0) (size 25.4 38.1)
+    (stroke (width 0.254) (type solid) (color 0 0 0 1))
+    (fill (type none))
+    (effects (font (size 2.794 2.794) (thickness 0.5588) bold (color 0 0 0 1)) (justify left top))
+  )
+  (text "TODO: \n- Add test points\n- De-page schematic" (at 100.33 124.46 0)
     (effects (font (size 1.27 1.27)) (justify left bottom))
   )
-  (symbol (lib_id "Mechanical:MountingHole") (at 190.5 76.2 0) (unit 1)
+  (symbol (lib_id "Mechanical:MountingHole") (at 196.85 76.2 0) (unit 1)
     (in_bom yes) (on_board yes) (dnp no) (fields_autoplaced)
-    (property "Reference" "H1" (at 193.04 74.93 0)
+    (property "Reference" "H1" (at 199.39 74.93 0)
       (effects (font (size 1.27 1.27)) (justify left))
     )
-    (property "Value" "MountingHole" (at 193.04 77.47 0)
+    (property "Value" "MountingHole" (at 199.39 77.47 0)
       (effects (font (size 1.27 1.27)) (justify left))
     )
-    (property "Footprint" "" (at 190.5 76.2 0)
+    (property "Footprint" "" (at 196.85 76.2 0)
       (effects (font (size 1.27 1.27)) hide)
     )
-    (property "Datasheet" "~" (at 190.5 76.2 0)
+    (property "Datasheet" "~" (at 196.85 76.2 0)
       (effects (font (size 1.27 1.27)) hide)
     )
@@
     )
   )
-  (symbol (lib_id "Mechanical:MountingHole") (at 190.5 88.9 0) (unit 1)
+  (symbol (lib_id "Mechanical:MountingHole") (at 196.85 88.9 0) (unit 1)
     (in_bom yes) (on_board yes) (dnp no) (fields_autoplaced)
-    (property "Reference" "H3" (at 193.04 87.63 0)
+    (property "Reference" "H3" (at 199.39 87.63 0)
       (effects (font (size 1.27 1.27)) (justify left))
     )
-    (property "Value" "MountingHole" (at 193.04 90.17 0)
+    (property "Value" "MountingHole" (at 199.39 90.17 0)
       (effects (font (size 1.27 1.27)) (justify left))
     )
-    (property "Footprint" "" (at 190.5 88.9 0)
+    (property "Footprint" "" (at 196.85 88.9 0)
       (effects (font (size 1.27 1.27)) hide)
     )
-    (property "Datasheet" "~" (at 190.5 88.9 0)
+    (property "Datasheet" "~" (at 196.85 88.9 0)
       (effects (font (size 1.27 1.27)) hide)
     )
@@
     )
   )
-  (symbol (lib_id "Mechanical:MountingHole") (at 190.5 95.25 0) (unit 1)
+  (symbol (lib_id "Mechanical:MountingHole") (at 196.85 95.25 0) (unit 1)
     (in_bom yes) (on_board yes) (dnp no) (fields_autoplaced)
-    (property "Reference" "H4" (at 193.04 93.98 0)
+    (property "Reference" "H4" (at 199.39 93.98 0)
       (effects (font (size 1.27 1.27)) (justify left))
     )
-    (property "Value" "MountingHole" (at 193.04 96.52 0)
+    (property "Value" "MountingHole" (at 199.39 96.52 0)
       (effects (font (size 1.27 1.27)) (justify left))
     )
-    (property "Footprint" "" (at 190.5 95.25 0)
+    (property "Footprint" "" (at 196.85 95.25 0)
       (effects (font (size 1.27 1.27)) hide)
     )
-    (property "Datasheet" "~" (at 190.5 95.25 0)
+    (property "Datasheet" "~" (at 196.85 95.25 0)
       (effects (font (size 1.27 1.27)) hide)
     )
@@
     )
   )
-  (symbol (lib_id "Mechanical:MountingHole") (at 190.5 82.55 0) (unit 1)
+  (symbol (lib_id "Mechanical:MountingHole") (at 196.85 82.55 0) (unit 1)
     (in_bom yes) (on_board yes) (dnp no) (fields_autoplaced)
-    (property "Reference" "H2" (at 193.04 81.28 0)
+    (property "Reference" "H2" (at 199.39 81.28 0)
       (effects (font (size 1.27 1.27)) (justify left))
     )
-    (property "Value" "MountingHole" (at 193.04 83.82 0)
+    (property "Value" "MountingHole" (at 199.39 83.82 0)
       (effects (font (size 1.27 1.27)) (justify left))
     )
-    (property "Footprint" "" (at 190.5 82.55 0)
+    (property "Footprint" "" (at 196.85 82.55 0)
       (effects (font (size 1.27 1.27)) hide)
     )
-    (property "Datasheet" "~" (at 190.5 82.55 0)
+    (property "Datasheet" "~" (at 196.85 82.55 0)
       (effects (font (size 1.27 1.27)) hide)
     )

Commit message: finished schematic v0.3
Parts:
- added D1: RST, symbol Device:LED
- added D2: PWR, symbol Device:LED
- added R1, R2: 1K, symbol Device:R
- added SW1: RESET, symbol Switch:SW_Push_Dual
- added U1: Raspberry-Pi-Pico, BeltFootprints:Raspberry-Pi-Pico, symbol Raspberry-Pi-Pico:Raspberry-Pi-Pico
Connections:
- new net: D2.1 (K), R2.1
- new net: D1.1 (K), R1.1
- new net +3.3V: D1.2 (A), U1.36 (3V3)
- new net +5V: D2.2 (A), U1.39 (V_{SYS})
- new net ADC0: U1.31 (GP_{26})
- new net GND: R2.2, SW1.1, SW1.3, U1.13 (GND), U1.18 (GND), U1.23 (GND), U1.28 (GND), U1.3 (GND), U1.38 (GND), U1.8 (GND)
- new net GNDA: U1.33 (AGND), U1.34 (GP_{28})
- new net SCL0: U1.7 (GP_{5})
- new net SDA0: U1.6 (GP_{4})
- new net ~{Reset}: R1.2, SW1.2, SW1.4, U1.37 (3V3_EN)
- no-connect marks 0 -> 25
Other:
- removed sheet Microcontroller
- note added: "ADC_{2} is tied to GNDA for ADC offset approximation."
- note added: "To improve ADC performance, add an external 3.0V shunt reference (such as LM4040) from ADC_V_{REF} to GNDA."
- note removed: "TODO: - Add test points - De-page schematic"
- moved on the sheet: H1, H2, H3, H4
