File: pcb/belt.kicad_pcb (KiCad board)
At the start: 2 copper layers, 19 parts, among them SW1 RESET, U1 Raspberry-Pi-Pico, U2 KP212K1409XTMA1, U3 AT30TS75A-SS8M

Commit message: completed initial layout
Parts:
- moved H4 127.9 mm to (174.0, 115.6)
- moved H2 115.9 mm to (174.0, 67.3)
- moved SW1 114.8 mm to (174.3, 78.1), turned to -90 degrees
- moved R4 111.4 mm to (172.1, 94.0), turned to 180 degrees
- moved R3 108.1 mm to (161.9, 99.1)
- moved R1 106.2 mm to (165.1, 74.9)
- moved D1 105.4 mm to (165.1, 71.1), turned to 90 degrees
- moved U1 105.3 mm to (146.1, 90.2)
- moved C1 104.9 mm to (174.0, 107.0), turned to -90 degrees
- moved U2 102.4 mm to (165.7, 109.5), turned to 90 degrees
- moved R5 98.1 mm to (161.9, 88.9)
- moved H3 88.0 mm to (118.1, 115.6)
- moved C2 81.7 mm to (163.5, 83.8)
- moved R6 72.5 mm to (127.0, 97.2), turned to 90 degrees
- moved R2 67.9 mm to (127.0, 74.9), turned to 180 degrees
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Routing:
- net +5V: track 0.00 -> 79.0 mm, vias 0 -> 3
- net +3.3V: track 0.00 -> 74.2 mm, vias 0 -> 2
- net /~{Reset}: track 0.00 -> 28.1 mm
- net GNDA: track 0.00 -> 13.7 mm, vias 0 -> 6
- net /ADC0: track 0.00 -> 11.3 mm
- net /SDA0: track 0.00 -> 11.0 mm, vias 0 -> 2
- net Net-(R3-Pad2): track 0.00 -> 10.2 mm
- net /SCL0: track 0.00 -> 9.44 mm
- net Net-(U3-ALERT): track 0.00 -> 8.24 mm
- net /Sensors/V_{baro_raw}: track 0.00 -> 7.67 mm
- net Net-(D2-K): track 0.00 -> 3.92 mm
- net Net-(D1-K): track 0.00 -> 3.81 mm
- added copper zone on F.Cu, net GND
- added copper zone on B.Cu, net GNDA
Other:
- board outline added: 63.5 x 55.9 mm
- rule pad_to_mask_clearance: 0 -> 0.0381
- board text added: "Adam Sher January 2024"
- board text added: "BELT"
- board text added: "Basic Electronics Learning Toolkit"
- board text added: "POWER"
- board text added: "RESET"
- board text added: "SYS OFF"
